File: ATMEGA328P Microcontroller.kicad_pcb (KiCad board)
At the start: 2 copper layers, 29 parts, among them J1 Conn_01x04_Pin, J2 Conn_01x04_Pin, J3 Conn_01x09_Pin, J4 Conn_02x03_Odd_Even, U1 24LC1025, U2 24LC1025, U3 ATmega328-P, U4 DS1337S_T_R, Y1 32.768 kHz, Y2 16MHz

Commit message: Updated block diagram and layout in progress
Parts:
- moved H3 116.7 mm to (100.2, 135.8)
- moved H1 104.4 mm to (100.2, 103.8)
- moved R4 99.2 mm to (119.1, 144.9)
- moved R3 99.1 mm to (129.8, 151.6), turned to 90 degrees
- moved R6 88.4 mm to (129.7, 156.0), turned to 90 degrees
- moved H4 80.2 mm to (151.5, 135.8)
- moved U4 79.0 mm to (121.7, 155.8)
- moved R2 75.7 mm to (133.7, 126.1)
- moved U3 70.5 mm to (145.1, 111.9), turned to -90 degrees
- moved U1 68.2 mm to (132.6, 133.6), turned to 90 degrees
- moved C3 67.8 mm to (111.6, 149.7)
- moved J4 67.6 mm to (99.8, 114.6)
- moved Y1 65.6 mm to (122.0, 149.5)
- moved R1 64.0 mm to (141.4, 126.0)
- moved H2 62.8 mm to (151.5, 103.8)
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Routing:
- net /SDA: track 0.00 -> 45.2 mm
- net /SCK: track 0.00 -> 32.2 mm
- net Net-(U3-XTAL1/PB6): track 0.00 -> 28.2 mm
- net Net-(BT1-+): track 0.00 -> 27.0 mm
- net /TX: track 0.00 -> 20.2 mm
- net Net-(U3-XTAL2/PB7): track 0.00 -> 19.5 mm
- net /D2: track 0.00 -> 11.8 mm
- net /D8: track 0.00 -> 11.4 mm
- net /D7: track 0.00 -> 11.4 mm
- net /D6: track 0.00 -> 11.4 mm
- net /D5: track 0.00 -> 11.4 mm
- net /D4: track 0.00 -> 10.1 mm
- net /D3: track 0.00 -> 10.1 mm
- net /RX: track 0.00 -> 8.85 mm
- net /RESET: track 0.00 -> 4.33 mm
Other:
- board outline added: 56.4 x 37.1 mm
